File: SMB-Lampe/kicad/SMB-Lampe.kicad_pcb (KiCad board)
At the start: 2 copper layers, 1 part, among them U1 MOUDLE-SEEEDUINO-XIAO-ESP32C3

Commit message: Beidseitige Platine Für hinteres Hinterbein
Routing:
- net (no net): track 0.00 -> 5.77 mm
Other:
- board outline added: 1.8 x 4.8 mm
