File: SMB-Lampe/kicad/Hinterbein_hinten_Seite1_LED-P/Hinterbein_hinten_Seite1_LED-P.kicad_sch (KiCad schematic)
At the start: 10 parts, among them J1 Conn_01x01_Pin, J2 Conn_01x01_Pin, J3 Conn_01x01_Pin, J5 Conn_01x01_Pin, J6 Conn_01x01_Pin

Commit message: vor Schaltplananpassung
Other:
- company: (none) -> IFM / Lukas Gulde
- title: (none) -> Projektaarbeit SMB-Lampe
Changed lines of the file:
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@@
 	(generator_version "9.0")
 	(paper "A4")
+	(title_block
+		(title "Projektaarbeit SMB-Lampe")
+		(date "2026-03-31")
+		(company "IFM / Lukas Gulde")
+	)
 	(text "Hinterbein hinten\nSeite 1 LED"
 		(exclude_from_sim no)
@@
 		)
 		(property "Value" "Conn_01x01_Pin"
-			(at 182.245 22.86 0)
-			(effects
-				(font
+			(at 182.372 22.352 0)
+			(effects
+				(font
