File: SMB-Lampe/kicad/Hinterbein_vorne_Seite2_LED-P/Hinterbein_vorne_Seite2_LED-P.kicad_pcb (KiCad board)
At the start: 2 copper layers, 10.7 x 29.2 mm, 5 parts

Commit message: Hinterbeine Geändert teilweiße Körper
Parts:
- C1: footprint Capacitor_SMD:C_0201_0603Metric -> Capacitor_SMD:C_0603_1608Metric_Pad1.08x0.95mm_HandSolder
- moved H3 0.28 mm to (154.8, 110.3)
Other:
- board text removed: "+"
- board text removed: "-"

Commit message: Alle Platinen sind fertig zur Fertigung
Aus diesem Stand folgt das erste fertig leuchtende Pferd
Parts:
- moved D1 0.11 mm to (151.5, 99.6)
Routing:
- net /+5V_IN_Hinterbein_vorne_Seite1: track 25.5 -> 25.0 mm
Other:
- board size 10.7 x 29.2 mm -> 11.5 x 29.2 mm

Commit message: Nachträgliche Änderungen für die Fertigung und Präsentation
Changed lines of the file:
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@@
 		(tags "LED RGB NeoPixel PLCC-4 5050")
 		(property "Reference" "D1"
-			(at 1.056812 -0.340071 108)
+			(at -1.571137 -3.675395 108)
 			(layer "F.SilkS")
 			(effects
@@
 		(at 154.85 110.35)
 		(property "Reference" "H3"
-			(at -0.13 -2.09 90)
-			(unlocked yes)
-			(layer "F.SilkS")
+			(at 0.65 -1.85 0)
+			(unlocked yes)
+			(layer "F.SilkS")
