File: SMB-Lampe/kicad/Hinterbein_vorne_Seite2_LED-P/Hinterbein_vorne_Seite2_LED-P.kicad_sch (KiCad schematic)
At the start: 0 parts

Commit message: Vorderes Hinterbein fertig
Alle Platinen sind fertig beschaltet
Parts:
- added C22: 100nF, Capacitor_SMD:C_0201_0603Metric, symbol Device:C
- added D22: WS2812B, LED_SMD:LED_WS2812B_PLCC4_5.0x5.0mm_P3.2mm, symbol LED:WS2812B
- added H24, H25, H26: MountingHole_Pad, Eigenen_Library:MountingHole D2 x d1 test, symbol Mechanical:MountingHole_Pad
Connections:
- new net +5V_IN_Hinterbein_vorne_Seite1: C22.1, D22.1 (VDD), H24.1
- new net Data_IN_Hinterbein_vorne_Seite1: D22.4 (DIN), H25.1
- new net GND: C22.2, D22.3 (VSS), H26.1
Other:
- note added: "Hinterbein vorne Seite 2 LED"

Commit message: Hinterbeine Geändert teilweiße Körper
Parts:
- C22: footprint Capacitor_SMD:C_0201_0603Metric -> Capacitor_SMD:C_0603_1608Metric_Pad1.08x0.95mm_HandSolder
Changed lines of the file:
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@@
 			)
 		)
-		(property "Footprint" "Capacitor_SMD:C_0201_0603Metric"
+		(property "Footprint" "Capacitor_SMD:C_0603_1608Metric_Pad1.08x0.95mm_HandSolder"
 			(at 78.4352 35.56 0)
 			(effects

Commit message: vor Schaltplananpassung
Other:
- note added: "LED Hinterbein vorne Seite 2"
- note removed: "Hinterbein vorne Seite 2 LED"
Changed lines of the file:
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@@
 	(generator_version "9.0")
 	(paper "A4")
-	(text "Hinterbein vorne\nSeite 2 LED"
+	(text "LED Hinterbein vorne\nSeite 2 "
 		(exclude_from_sim no)
 		(at 89.408 74.676 0)

Commit message: Änderungen für Dokumentation
Other:
- company: (none) -> IFM / Lukas Gulde
- title: (none) -> Projektaarbeit SMB-Lampe
Changed lines of the file:
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@@
 	(generator_version "9.0")
 	(paper "A4")
+	(title_block
+		(title "Projektaarbeit SMB-Lampe")
+		(date "2026-03-31")
+		(company "IFM / Lukas Gulde")
+	)
 	(text "LED Hinterbein vorne\nSeite 2 "
 		(exclude_from_sim no)
