File: SMB-Lampe/kicad/Körper_Seite1/Körper_Seite1.kicad_pcb (KiCad board)
At the start: 2 copper layers, 135.9 x 93.9 mm, 32 parts, among them J1 Conn_01x01_Pin, J2 Conn_01x01_Pin, J3 Conn_01x01_Pin

Commit message: vor Schaltplananpassung
Changed lines of the file:
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@@
 		(at 110.5 105.5)
 		(property "Reference" "H3"
-			(at 0 -1 0)
+			(at 0.1 -1.9 0)
 			(unlocked yes)
 			(layer "F.SilkS")
@@
 		(at 114.5 105.5)
 		(property "Reference" "H1"
-			(at 0 -1 0)
-			(unlocked yes)
-			(layer "F.SilkS")
+			(at 0.1 -1.9 0)
+			(unlocked yes)
+			(layer "F.SilkS")
