File: SMB-Lampe/kicad/Körper_Seite1/Körper_Seite1.kicad_sch (KiCad schematic)
At the start: 28 parts, among them J7 Conn_01x01_Pin, J8 Conn_01x01_Pin, J9 Conn_01x01_Pin

Commit message: Änderungen für Dokumentation
Other:
- note added: "+5V für LED 13-15,20 Seite 2 (Platinreferenc 2-4,9)"
- note added: "+5V für LED 16-19 Seite 2 (Platinreferenc 5-8)"
- note added: "GND für LED 13-15,20 Seite 2 (Platinreferenc 2-4,9)"
- note added: "GND für LED 7-10 Seite1 (Platinreferenc 5-8)"
- note removed: "+5V für LED 2-4,9 Seite 2"
- note removed: "+5V für LED 5-8 Seite 2"
- note removed: "GND für LED 2-4,9 Seite 2"
- note removed: "GND für LED 5-8 Seite 1"
- company: (none) -> IFM / Lukas Gulde
- title: (none) -> Projektaarbeit SMB-Lampe
Changed lines of the file:
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@@
 	(generator_version "9.0")
 	(paper "A4")
-	(text "+5V für LED 5-8 Seite 2"
+	(title_block
+		(title "Projektaarbeit SMB-Lampe")
+		(date "2026-03-31")
+		(company "IFM / Lukas Gulde")
+	)
+	(text "GND für LED 7-10 Seite1\n(Platinreferenc 5-8)\n"
 		(exclude_from_sim no)
-		(at 256.286 95.504 0)
+		(at 31.75 72.39 0)
 		(effects
 			(font
@@
 		)
 	)
-	(text "GND für LED 2-4,9 Seite 2"
+	(text "+5V für LED 16-19 Seite 2\n(Platinreferenc 5-8)"
 		(exclude_from_sim no)
-		(at 260.858 151.638 0)
+		(at 258.318 96.52 0)
 		(effects
 			(font
@@
 		)
 	)
-	(text "GND für LED 5-8 Seite 1"
+	(text "+5V für LED 13-15,20 Seite 2\n(Platinreferenc 2-4,9)"
 		(exclude_from_sim no)
-		(at 33.528 71.628 0)
+		(at 259.588 89.408 0)
 		(effects
 			(font
@@
 		)
 	)
-	(text "+5V für LED 2-4,9 Seite 2"
+	(text "GND für LED 13-15,20 Seite 2\n(Platinreferenc 2-4,9)"
 		(exclude_from_sim no)
-		(at 257.302 90.678 0)
+		(at 262.89 153.67 0)
 		(effects
 			(font
