File: SMB-Lampe/kicad/Körper_Seite2/Körper_Seite2.kicad_sch (KiCad schematic)
At the start: 28 parts, among them J16 Conn_01x01_Pin, J17 Conn_01x01_Pin, J18 Conn_01x01_Pin

Commit message: vor Schaltplananpassung
Other:
- note added: "+5V für LED 13-15,20 Seite 2 (Platinreferenc 2-4,9)"
- note added: "+5V für LED 16-19 Seite 2 (Platinreferenc 5-8)"
- note added: "GND für LED 13-15,20 Seite 2 (Platinreferenc 2-4,9)"
- note added: "GND für LED 7-10 Seite1 (Platinreferenc 5-8)"
- note removed: "+5V für LED 2-4,9 Seite 2"
- note removed: "+5V für LED 5-8 Seite 2"
- note removed: "GND für LED 5-8 Seite 2"
- note removed: "GND für LED 5-8 Seite1"
- company: (none) -> IFM / Lukas Gulde
- title: (none) -> Projektaarbeit SMB-Lampe
- moved on the sheet: H10, H11, H12, H14, H19, H20
Changed lines of the file:
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@@
 	(generator_version "9.0")
 	(paper "A4")
-	(text "GND für LED 5-8 Seite 2"
+	(title_block
+		(title "Projektaarbeit SMB-Lampe")
+		(date "2026-03-31")
+		(company "IFM / Lukas Gulde")
+	)
+	(text "GND für LED 13-15,20 Seite 2\n(Platinreferenc 2-4,9)"
 		(exclude_from_sim no)
-		(at 27.178 81.788 0)
+		(at 27.178 81.026 0)
 		(effects
 			(font
@@
 		)
 	)
-	(text "GND für LED 5-8 Seite1"
+	(text "GND für LED 7-10 Seite1\n(Platinreferenc 5-8)\n"
 		(exclude_from_sim no)
 		(at 270.764 146.558 0)
@@
 		)
 	)
-	(text "+5V für LED 2-4,9 Seite 2"
+	(text "+5V für LED 13-15,20 Seite 2\n(Platinreferenc 2-4,9)"
 		(exclude_from_sim no)
-		(at 27.178 48.768 0)
+		(at 28.448 49.53 0)
 		(effects
 			(font
@@
 		)
 	)
-	(text "+5V für LED 5-8 Seite 2"
+	(text "+5V für LED 16-19 Seite 2\n(Platinreferenc 5-8)"
 		(exclude_from_sim no)
-		(at 27.178 43.688 0)
+		(at 27.178 43.942 0)
 		(effects
 			(font
@@
 	)
 	(junction
-		(at 63.5 76.2)
+		(at 69.85 76.2)
 		(diameter 0)
 		(color 0 0 0 0)
@@
 	)
 	(junction
-		(at 63.5 43.18)
+		(at 69.85 43.18)
 		(diameter 0)
 		(color 0 0 0 0)
 	)
 	(junction
-		(at 63.5 38.1)
+		(at 69.85 38.1)
 		(diameter 0)
 		(color 0 0 0 0)
@@
 	)
 	(junction
-		(at 63.5 57.15)
+		(at 69.85 57.15)
 		(diameter 0)
 		(color 0 0 0 0)
@@
 	(wire
 		(pts
-			(xy 63.5 38.1) (xy 63.5 43.18)
+			(xy 69.85 38.1) (xy 69.85 43.18)
 		)
 		(stroke
@@
 	(wire
 		(pts
-			(xy 63.5 76.2) (xy 63.5 81.28)
+			(xy 69.85 76.2) (xy 69.85 81.28)
 		)
 		(stroke
@@
 	(wire
 		(pts
-			(xy 63.5 38.1) (xy 77.47 38.1)
+			(xy 69.85 38.1) (xy 77.47 38.1)
 		)
 		(stroke
@@
 	(wire
 		(pts
-			(xy 63.5 57.15) (xy 81.28 57.15)
+			(xy 69.85 57.15) (xy 81.28 57.15)
 		)
 		(stroke
@@
 	(wire
 		(pts
-			(xy 63.5 43.18) (xy 63.5 48.26)
+			(xy 69.85 43.18) (xy 69.85 48.26)
 		)
 		(stroke
@@
 	(wire
 		(pts
-			(xy 63.5 76.2) (xy 88.9 76.2)
+			(xy 69.85 76.2) (xy 88.9 76.2)
 		)
 		(stroke
@@
 	(wire
 		(pts
-			(xy 50.8 38.1) (xy 63.5 38.1)
+			(xy 57.15 38.1) (xy 69.85 38.1)
 		)
 		(stroke
@@
 	(wire
 		(pts
-			(xy 50.8 57.15) (xy 63.5 57.15)
+			(xy 57.15 57.15) (xy 69.85 57.15)
 		)
 		(stroke
@@
 	(wire
 		(pts
-			(xy 50.8 76.2) (xy 63.5 76.2)
+			(xy 57.15 76.2) (xy 69.85 76.2)
 		)
 		(stroke
@@
 	(hierarchical_label "GND_IN_Körper_Seite1"
 		(shape input)
-		(at 50.8 76.2 180)
+		(at 57.15 76.2 180)
 		(effects
 			(font
@@
 	(hierarchical_label "+5V_IN_Körper_Seite1"
 		(shape input)
-		(at 50.8 38.1 180)
+		(at 57.15 38.1 180)
 		(effects
 			(font
@@
 	(hierarchical_label "Data_IN_Körper_Seite1"
 		(shape input)
-		(at 50.8 57.15 180)
+		(at 57.15 57.15 180)
 		(effects
 			(font
@@
 	(symbol
 		(lib_id "Mechanical:MountingHole_Pad")
-		(at 60.96 81.28 90)
+		(at 67.31 81.28 90)
 		(unit 1)
 		(exclude_from_sim no)
@@
 		(dnp no)
 		(property "Reference" "H20"
-			(at 49.276 80.01 90)
+			(at 53.34 80.01 90)
 			(effects
 				(font
@@
 		)
 		(property "Value" "MountingHole_Pad"
-			(at 49.276 82.55 90)
+			(at 53.34 82.55 90)
 			(effects
 				(font
@@
 		)
 		(property "Footprint" "Eigenen_Library:MountingHole D2 x d1 test"
-			(at 60.96 81.28 0)
+			(at 67.31 81.28 0)
 			(effects
 				(font
@@
 		)
 		(property "Datasheet" "~"
-			(at 60.96 81.28 0)
+			(at 67.31 81.28 0)
 			(effects
 				(font
@@
 		)
 		(property "Description" "Mounting Hole with connection"
-			(at 60.96 81.28 0)
+			(at 67.31 81.28 0)
 			(effects
 				(font
@@
 	(symbol
 		(lib_id "Mechanical:MountingHole_Pad")
-		(at 60.96 57.15 90)
+		(at 67.31 57.15 90)
 		(unit 1)
 		(exclude_from_sim no)
@@
 		(dnp no)
 		(property "Reference" "H11"
-			(at 59.944 60.706 90)
+			(at 66.294 60.706 90)
 			(effects
 				(font
@@
 		)
 		(property "Value" "MountingHole_Pad"
-			(at 59.944 63.246 90)
+			(at 66.294 63.246 90)
 			(effects
 				(font
@@
 		)
 		(property "Footprint" "Eigenen_Library:MountingHole D2 x d1 test"
-			(at 60.96 57.15 0)
+			(at 67.31 57.15 0)
 			(effects
 				(font
@@
 		)
 		(property "Datasheet" "~"
-			(at 60.96 57.15 0)
+			(at 67.31 57.15 0)
 			(effects
 				(font
@@
 		)
 		(property "Description" "Mounting Hole with connection"
-			(at 60.96 57.15 0)
+			(at 67.31 57.15 0)
 			(effects
 				(font
@@
 	(symbol
 		(lib_id "Mechanical:MountingHole_Pad")
-		(at 60.96 48.26 90)
+		(at 67.31 48.26 90)
 		(unit 1)
 		(exclude_from_sim no)
@@
 		(dnp no)
 		(property "Reference" "H19"
-			(at 49.276 46.99 90)
+			(at 54.356 46.99 90)
 			(effects
 				(font
@@
 		)
 		(property "Value" "MountingHole_Pad"
-			(at 49.276 49.53 90)
+			(at 54.356 49.53 90)
 			(effects
 				(font
@@
 		)
 		(property "Footprint" "Eigenen_Library:MountingHole D2 x d1 test"
-			(at 60.96 48.26 0)
+			(at 67.31 48.26 0)
 			(effects
 				(font
@@
 		)
 		(property "Datasheet" "~"
-			(at 60.96 48.26 0)
+			(at 67.31 48.26 0)
 			(effects
 				(font
@@
 		)
 		(property "Description" "Mounting Hole with connection"
-			(at 60.96 48.26 0)
+			(at 67.31 48.26 0)
 			(effects
 				(font
@@
 	(symbol
 		(lib_id "Mechanical:MountingHole_Pad")
-		(at 60.96 43.18 90)
+		(at 67.31 43.18 90)
 		(unit 1)
 		(exclude_from_sim no)
@@
 		(dnp no)
 		(property "Reference" "H14"
-			(at 49.276 41.91 90)
+			(at 54.356 41.91 90)
 			(effects
 				(font
@@
 		)
 		(property "Value" "MountingHole_Pad"
-			(at 49.276 44.45 90)
+			(at 54.356 44.45 90)
 			(effects
 				(font
@@
 		)
 		(property "Footprint" "Eigenen_Library:MountingHole D2 x d1 test"
-			(at 60.96 43.18 0)
+			(at 67.31 43.18 0)
 			(effects
 				(font
@@
 		)
 		(property "Datasheet" "~"
-			(at 60.96 43.18 0)
+			(at 67.31 43.18 0)
 			(effects
 				(font
@@
 		)
 		(property "Description" "Mounting Hole with connection"
-			(at 60.96 43.18 0)
+			(at 67.31 43.18 0)
 			(effects
 				(font
@@
 	(symbol
 		(lib_id "Mechanical:MountingHole_Pad")
-		(at 60.96 38.1 90)
+		(at 67.31 38.1 90)
 		(unit 1)
 		(exclude_from_sim no)
@@
 		(fields_autoplaced yes)
 		(property "Reference" "H10"
-			(at 59.69 31.75 90)
+			(at 66.04 31.75 90)
 			(effects
 				(font
@@
 		)
 		(property "Value" "MountingHole_Pad"
-			(at 59.69 34.29 90)
+			(at 66.04 34.29 90)
 			(effects
 				(font
@@
 		)
 		(property "Footprint" "Eigenen_Library:MountingHole D2 x d1 test"
-			(at 60.96 38.1 0)
+			(at 67.31 38.1 0)
 			(effects
 				(font
@@
 		)
 		(property "Datasheet" "~"
-			(at 60.96 38.1 0)
+			(at 67.31 38.1 0)
 			(effects
 				(font
@@
 		)
 		(property "Description" "Mounting Hole with connection"
-			(at 60.96 38.1 0)
+			(at 67.31 38.1 0)
 			(effects
 				(font
@@
 	(symbol
 		(lib_id "Mechanical:MountingHole_Pad")
-		(at 60.96 76.2 90)
+		(at 67.31 76.2 90)
 		(unit 1)
 		(exclude_from_sim no)
@@
 		(fields_autoplaced yes)
 		(property "Reference" "H12"
-			(at 59.69 69.85 90)
+			(at 66.04 69.85 90)
 			(effects
 				(font
@@
 		)
 		(property "Value" "MountingHole_Pad"
-			(at 59.69 72.39 90)
+			(at 66.04 72.39 90)
 			(effects
 				(font
@@
 		)
 		(property "Footprint" "Eigenen_Library:MountingHole D2 x d1 test"
-			(at 60.96 76.2 0)
+			(at 67.31 76.2 0)
 			(effects
 				(font
@@
 		)
 		(property "Datasheet" "~"
-			(at 60.96 76.2 0)
+			(at 67.31 76.2 0)
 			(effects
 				(font
@@
 		)
 		(property "Description" "Mounting Hole with connection"
-			(at 60.96 76.2 0)
+			(at 67.31 76.2 0)
 			(effects
 				(font
