File: SMB-Lampe/kicad/Körper_Seite2/Körper_Seite2.kicad_sch (KiCad schematic)
At the start: 28 parts, among them J16 Conn_01x01_Pin, J17 Conn_01x01_Pin, J18 Conn_01x01_Pin

Commit message: Änderungen für Dokumentation
Connections:
- net Data renamed Data2
Changed lines of the file:
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@@
 	(text "GND für LED 13-15,20 Seite 2\n(Platinreferenc 2-4,9)"
 		(exclude_from_sim no)
-		(at 27.178 81.026 0)
+		(at 28.194 81.534 0)
 		(effects
 			(font
@@
 		)
 	)
-	(global_label "Data"
+	(global_label "Data2"
 		(shape input)
 		(at 25.4 120.65 180)
@@
 		)
 		(property "Intersheetrefs" "${INTERSHEET_REFS}"
-			(at 18.1211 120.65 0)
+			(at 16.9116 120.65 0)
 			(effects
 				(font
@@
 		)
 	)
-	(global_label "Data"
+	(global_label "Data2"
 		(shape input)
 		(at 266.7 57.15 0)
@@
 		)
 		(property "Intersheetrefs" "${INTERSHEET_REFS}"
-			(at 273.9789 57.15 0)
+			(at 275.1884 57.15 0)
 			(effects
 				(font
