File: SMB-Lampe/kicad/Hinterbein_hinten_Seite2_LED-P/Hinterbein_hinten_Seite2_LED-P.kicad_sch (KiCad schematic)
At the start: 0 parts

Commit message: Hinterbein Seite 1/2 erstellt
Anschlüsse zwischen den Platinen mit MountingHoles. Eigenes MountingHole Erstellt
Parts:
- added C2: 100nF, Capacitor_SMD:C_0201_0603Metric, symbol Device:C
- added D2: WS2812B, LED_SMD:LED_WS2812B_PLCC4_5.0x5.0mm_P3.2mm, symbol LED:WS2812B
- added H4, H5, H6: MountingHole_Pad, Eigenen_Library:MountingHole D2,5 x d1 test, symbol Mechanical:MountingHole_Pad
- added J22: Conn_01x01_Pin, TestPoint:TestPoint_Pad_2.0x2.0mm, symbol Connector:Conn_01x01_Pin
Connections:
- new net +5V_IN_Hinterbein_hinten_Seite1: C2.1, D2.1 (VDD), H4.1
- new net Data_IN_Hinterbein_hinten_Seite1: D2.4 (DIN), H5.1
- new net Data_OUT_Körper_Seite1: D2.2 (DOUT), J22.1 (Pin_1)
- new net GND: C2.2, D2.3 (VSS), H6.1
Other:
- note added: "Hinterbeein hinten Seite 2 LED"

Commit message: Hinterbein Hinten fertig
Seite 1 und Seite 2 von Hinterbein hinten Sind fertig
Parts:
- H4, H5, H6: footprint Eigenen_Library:MountingHole D2,5 x d1 test -> Eigenen_Library:MountingHole D2 x d1 test
Changed lines of the file:
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@@
 			)
 		)
-		(property "Footprint" "Eigenen_Library:MountingHole D2,5 x d1 test"
+		(property "Footprint" "Eigenen_Library:MountingHole D2 x d1 test"
 			(at 60.96 44.45 0)
 			(effects
@@
 			)
 		)
-		(property "Footprint" "Eigenen_Library:MountingHole D2,5 x d1 test"
+		(property "Footprint" "Eigenen_Library:MountingHole D2 x d1 test"
 			(at 60.96 63.5 0)
 			(effects
@@
 			)
 		)
-		(property "Footprint" "Eigenen_Library:MountingHole D2,5 x d1 test"
+		(property "Footprint" "Eigenen_Library:MountingHole D2 x d1 test"
 			(at 60.96 25.4 0)
 			(effects

Commit message: Vorderseite Platine Körper Seite 1 fertig
zwei GND Verbindungen fehlen noch
Other:
- note added: "Hinterbein hinten Seite 2 LED"
- note removed: "Hinterbeein hinten Seite 2 LED"
Changed lines of the file:
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@@
 	(generator_version "9.0")
 	(paper "A4")
-	(text "Hinterbeein hinten\nSeite 2 LED"
+	(text "Hinterbein hinten\nSeite 2 LED"
 		(exclude_from_sim no)
 		(at 89.408 74.676 0)

Commit message: Hinterbeine Geändert teilweiße Körper
Parts:
- C1: renamed from C2; footprint Capacitor_SMD:C_0201_0603Metric -> Capacitor_SMD:C_0603_1608Metric_Pad1.08x0.95mm_HandSolder
- renumbered D2 to D1, H4 to H1, H5 to H2, H6 to H3, J22 to J1
Changed lines of the file:
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@@
 		(dnp no)
 		(fields_autoplaced yes)
-		(property "Reference" "C2"
+		(property "Reference" "C1"
 			(at 81.28 30.4799 0)
 			(effects
@@
 			)
 		)
-		(property "Footprint" "Capacitor_SMD:C_0201_0603Metric"
+		(property "Footprint" "Capacitor_SMD:C_0603_1608Metric_Pad1.08x0.95mm_HandSolder"
 			(at 78.4352 35.56 0)
 			(effects
@@
 				)
 			)
+			(project "Hinterbein_hinten_Seite2_LED-P"
+				(path "/83b66c53-7ffd-447e-9eb8-b29b3c8d8322"
+					(reference "C1")
+					(unit 1)
+				)
+			)
 		)
 	)
@@
 		(dnp no)
 		(fields_autoplaced yes)
-		(property "Reference" "#PWR0103"
+		(property "Reference" "#PWR0102"
 			(at 63.5 69.85 0)
 			(effects
@@
 				)
 			)
+			(project "Hinterbein_hinten_Seite2_LED-P"
+				(path "/83b66c53-7ffd-447e-9eb8-b29b3c8d8322"
+					(reference "#PWR0102")
+					(unit 1)
+				)
+			)
 		)
 	)
@@
 		(dnp no)
 		(fields_autoplaced yes)
-		(property "Reference" "H5"
+		(property "Reference" "H2"
 			(at 59.69 38.1 90)
 			(effects
@@
 				)
 			)
+			(project "Hinterbein_hinten_Seite2_LED-P"
+				(path "/83b66c53-7ffd-447e-9eb8-b29b3c8d8322"
+					(reference "H2")
+					(unit 1)
+				)
+			)
 		)
 	)
@@
 		(dnp no)
 		(fields_autoplaced yes)
-		(property "Reference" "H6"
+		(property "Reference" "H3"
 			(at 59.69 57.15 90)
 			(effects
@@
 				)
 			)
+			(project "Hinterbein_hinten_Seite2_LED-P"
+				(path "/83b66c53-7ffd-447e-9eb8-b29b3c8d8322"
+					(reference "H3")
+					(unit 1)
+				)
+			)
 		)
 	)
@@
 		(dnp no)
 		(fields_autoplaced yes)
-		(property "Reference" "H4"
+		(property "Reference" "H1"
 			(at 59.69 19.05 90)
 			(effects
@@
 				)
 			)
+			(project "Hinterbein_hinten_Seite2_LED-P"
+				(path "/83b66c53-7ffd-447e-9eb8-b29b3c8d8322"
+					(reference "H1")
+					(unit 1)
+				)
+			)
 		)
 	)
@@
 				)
 			)
+			(project "Hinterbein_hinten_Seite2_LED-P"
+				(path "/83b66c53-7ffd-447e-9eb8-b29b3c8d8322"
+					(reference "#PWR0101")
+					(unit 1)
+				)
+			)
 		)
 	)
@@
 		(dnp no)
 		(fields_autoplaced yes)
-		(property "Reference" "J22"
+		(property "Reference" "J1"
 			(at 131.445 39.37 0)
 			(effects
@@
 				)
 			)
+			(project "Hinterbein_hinten_Seite2_LED-P"
+				(path "/83b66c53-7ffd-447e-9eb8-b29b3c8d8322"
+					(reference "J1")
+					(unit 1)
+				)
+			)
 		)
 	)
@@
 		(on_board yes)
 		(dnp no)
-		(property "Reference" "D2"
+		(property "Reference" "D1"
 			(at 100.33 38.0298 0)
 			(effects
@@
 				)
 			)
-		)
-	)
+			(project "Hinterbein_hinten_Seite2_LED-P"
+				(path "/83b66c53-7ffd-447e-9eb8-b29b3c8d8322"
+					(reference "D1")
+					(unit 1)
+				)
+			)
+		)
+	)
+	(sheet_instances
+		(path "/"
+			(page "1")
+		)
+	)
+	(embedded_fonts no)
 )

Commit message: Hauptplatine fertig
Hauptplatine mit ESP Levelshifter und Screwsockets
Parts:
- renumbered C1 to C2, D1 to D2, H1 to H4, H2 to H5, H3 to H6, J1 to J22
Changed lines of the file:
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@@
 		(dnp no)
 		(fields_autoplaced yes)
-		(property "Reference" "C1"
+		(property "Reference" "C2"
 			(at 81.28 30.4799 0)
 			(effects
@@
 		(dnp no)
 		(fields_autoplaced yes)
-		(property "Reference" "#PWR0102"
+		(property "Reference" "#PWR0103"
 			(at 63.5 69.85 0)
 			(effects
@@
 		(dnp no)
 		(fields_autoplaced yes)
-		(property "Reference" "H2"
+		(property "Reference" "H5"
 			(at 59.69 38.1 90)
 			(effects
@@
 		(dnp no)
 		(fields_autoplaced yes)
-		(property "Reference" "H3"
+		(property "Reference" "H6"
 			(at 59.69 57.15 90)
 			(effects
@@
 		(dnp no)
 		(fields_autoplaced yes)
-		(property "Reference" "H1"
+		(property "Reference" "H4"
 			(at 59.69 19.05 90)
 			(effects
@@
 		(dnp no)
 		(fields_autoplaced yes)
-		(property "Reference" "J1"
+		(property "Reference" "J22"
 			(at 131.445 39.37 0)
 			(effects
@@
 		(on_board yes)
 		(dnp no)
-		(property "Reference" "D1"
+		(property "Reference" "D2"
 			(at 100.33 38.0298 0)
 			(effects

Commit message: Änderungen für Dokumentation
Other:
- company: (none) -> IFM / Lukas Gulde
- title: (none) -> Projektaarbeit SMB-Lampe
Changed lines of the file:
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@@
 	(generator_version "9.0")
 	(paper "A4")
+	(title_block
+		(title "Projektaarbeit SMB-Lampe")
+		(date "2026-03-31")
+		(company "IFM / Lukas Gulde")
+	)
 	(text "Hinterbein hinten\nSeite 2 LED"
 		(exclude_from_sim no)
